File: boardv1.0.sch (EAGLE design)
At the start: 60 parts, among them IC3 LM1117, J2 ICSP, J3 POWER_JACKSUPER_BOMB_DIGITY, Q1 1A/60V/500mΩ, Q2 2N7002PW, U1 FT231XS, U2 MIC5205, U4 ATMEGA328P_TQFP, Y1 16MHz

Commit message: Bluetooth added
Parts:
- removed JP10: JP10, SparkFun-Connectors:M08SMD-COMBO
- added C11, C25: 0.1µF, microbuilder:CAP_CERAMIC0805-NOOUTLINE
- added C16: 2.2nF, microbuilder:CAP_CERAMIC_0402
- added C17: 0.1uF, microbuilder:CAP_CERAMIC0805-NOOUTLINE
- added C18: 33nF, microbuilder:CAP_CERAMIC0805-NOOUTLINE
- added C19, C20, C21, C22: 15pF, microbuilder:CAP_CERAMIC0805-NOOUTLINE
- added C23: 1µF, microbuilder:CAP_CERAMIC0805-NOOUTLINE
- added C24: 1nF, microbuilder:CAP_CERAMIC_0603
- added C26: 10µF, microbuilder:CAP_CERAMIC0805-NOOUTLINE
- added C28: 1.8pF, microbuilder:CAP_CERAMIC_0402MP
- added C29: 1.2pF, microbuilder:CAP_CERAMIC_0402MP
- added C30: 1.5pF, microbuilder:CAP_CERAMIC_0402MP
- added FB1: MMZ1608B121C, microbuilder:FERRITE0805
- added FID3: FIDUCIAL"", microbuilder:FIDUCIAL""
- added L1: 8.2nH, microbuilder:INDUCTOR_0402
- added L2: 5.6nH, microbuilder:INDUCTOR_0402
- added L3: 3.9nH, microbuilder:INDUCTOR_0402
- added L4: 10µH, microbuilder:INDUCTOR_0603
- added L5: 15nH, microbuilder:INDUCTOR_0603
- added R18: 22K, microbuilder:RESISTOR_0805MP
- added R20: 10k, SparkFun-Resistors:10KOHM-0603-1/10W-1%
- added U$37: (no value), microbuilder:ANTENNA_PCBNRF8001_1.6MM
- added U3: nRF8001, microbuilder:NRF8001
- added U6: 74HC4050D, microbuilder:74HC4050DTSSOP
- added Y2: 16MHz, microbuilder:CRYSTAL3.2X2.5
- added Y3: FC-255 32.7680K-A3, microbuilder:CRYSTAL8.0X3.8
- R16: value 1k -> 4.7k
Connections:
- removed net DP9: JP4.2, U4.PB1(OC1A)
- new net ACTIVE: U3A.ACTIVE
- new net AVDD: C11.1, C23.1, C24.1, FB1.P$2, L5.2, U3A.AVDD@1, U3A.AVDD@2, U3A.AVDD@3
- new net DP3: U4.PD3(INT1)
- new net DP4: U4.PD4(XCK/T0)
- new net DP5: R12.1, U4.PD5(T1)
- new net MOSI_3V: U3A.MOSI, U6.1Y
- new net N$1: C16.1, L2.2, U3A.VDD_PA
- new net N$11: C20.1, U3A.XC1, Y2.2
- new net N$12: C19.1, U3A.XC2, Y2.1
- new net N$13: L4.1, U3A.DCC
- new net N$14: R18.1, U3A.IREF
- new net N$16: L4.2, L5.1
- new net N$17: L1.2, L3.1, U3A.ANT2
- new net N$18: L1.1, L2.1, U3A.ANT1
- new net N$19: C28.2, L3.2
- new net N$20: C28.1, C29.2, C30.2, U$37.P$1
- new net N$22: C21.2, U3A.XL2, Y3.1
- new net N$23: C22.2, U3A.XL1, Y3.2
- new net N$5: C18.1, U3A.DEC2
- new net N$9: C17.1, U3A.DEC1
- new net RDYN: R20.1, U3A.RDYN, U4.PD2(INT0)
- new net REQN: U4.PB2(SS/OC1B), U6.2A
- new net REQN_3V: U3A.REQN, U6.2Y
- new net RESET_3V: U3A.RESET, U6.4Y
- new net SCK_3V: U3A.SCK, U6.3Y
- net 3.3V: now also C25.1, C26.1, FB1.P$1, R20.2, U3A.VDD@1, U3A.VDD@2, U6.VCC; no longer JP10.5
- net 5V: no longer JP10.4, JP10.7
- net DP6: now also R1.2; no longer JP3.2, R16.1
- net DP7: now also JP3.2, R16.1; no longer R12.1
- net DP8: now also JP4.2; no longer R1.2
- net GND: now also C11.2, C16.2, C17.2, C18.2, C19.2, C20.2, C21.1, C22.1, C23.2, C24.2, C25.2, C26.2, C29.1, C30.1, R18.2, U3-SLUG.TP, U3A.VSS@1, U3A.VSS@2, U3A.VSS@3, U3A.VSS@4, U3A.VSS@5, U3A.VSS@6, U6.GND; no longer JP10.2, JP10.3
- net MISO: now also U3A.MISO, U4.PB4(MISO)
- net MOSI: now also U4.PB3(MOSI/OC2), U6.1A
- net RESET: now also U4.PB1(OC1A); no longer JP10.6
- net SCK: now also U4.PB5(SCK), U6.3A, U6.4A
- net VIN: no longer JP10.1
Other:
- note added: "Analog Supply Filtering"
- note added: "SPI MODE 0"
- note added: "but RDYN and REQN"
- note added: "replace CS"
